File: Rev.2/CAD/37c3PCBLEDC100R_Rev.2.kicad_pcb (KiCad board)
At the start: 2 copper layers, 100 x 100 mm, 25 parts, among them Q1 BSS138, U1 WeMos_D1_mini

Commit message: Updated Libs & changes on Top Silkscreen
Parts:
- D1, D2, D3, D4, D5, D6, D7, D8: value WS2812B -> WS2812D-F5
- renumbered TP1 to DIN, TP2 to DOUT
Connections:
- D1 pad 1: +5V -> Net-(D1-DOUT)
- D1 pad 2: Net-(D1-DOUT) -> +5V
- D2 pad 1: +5V -> Net-(D2-VDD)
- D2 pad 2: Net-(D2-DOUT) -> +5V
- D3 pad 1: +5V -> Net-(D3-VDD)
- D3 pad 2: Net-(D3-DOUT) -> +5V
- D3 pad 4: Net-(D2-DOUT) -> Net-(D2-VDD)
- D4 pad 1: +5V -> Net-(D4-VDD)
- D4 pad 2: Net-(D4-DOUT) -> +5V
- D4 pad 4: Net-(D3-DOUT) -> Net-(D3-VDD)
- D5 pad 1: +5V -> Net-(D5-VDD)
- D5 pad 2: Net-(D5-DOUT) -> +5V
- D5 pad 4: Net-(D4-DOUT) -> Net-(D4-VDD)
- D6 pad 1: +5V -> Net-(D6-VDD)
- D6 pad 2: Net-(D6-DOUT) -> +5V
- D6 pad 4: Net-(D5-DOUT) -> Net-(D5-VDD)
- D7 pad 1: +5V -> Net-(D7-VDD)
- D7 pad 2: Net-(D7-DOUT) -> +5V
- D7 pad 4: Net-(D6-DOUT) -> Net-(D6-VDD)
- D8 pad 1: +5V -> /Dout
- D8 pad 2: /Dout -> +5V
- D8 pad 4: Net-(D7-DOUT) -> Net-(D7-VDD)
Routing:
- net Net-(D3-VDD): track 0.00 -> 33.7 mm
- net Net-(D3-DOUT): track 33.7 -> 0.00 mm
- net Net-(D2-VDD): track 0.00 -> 32.6 mm
- net Net-(D2-DOUT): track 32.6 -> 0.00 mm
- net Net-(D7-VDD): track 0.00 -> 32.3 mm
- net Net-(D7-DOUT): track 32.3 -> 0.00 mm
- net Net-(D5-VDD): track 0.00 -> 32.3 mm
- net Net-(D5-DOUT): track 32.3 -> 0.00 mm
- net Net-(D6-VDD): track 0.00 -> 32.3 mm
- net Net-(D6-DOUT): track 32.3 -> 0.00 mm
- net Net-(D4-VDD): track 0.00 -> 31.9 mm
- net Net-(D4-DOUT): track 31.9 -> 0.00 mm
Other:
- board text added: "37c3PCBLEDC100R Rev.2"
- board text removed: "Untersetzer 0.1 Rev.2"
