File: Rev.2/CAD/37c3PCBLEDC100R_Rev.2.kicad_sch (KiCad schematic)
At the start: 20 parts, among them Q1 BSS138, U1 WeMos_D1_mini

Commit message: Updated Libs & changes on Top Silkscreen
Parts:
- D1, D2, D3, D4, D5, D6, D7, D8: value WS2812B -> WS2812D-F5; symbol LED:WS2812B -> WS2812D-F5-1261:WS2812D-F5-1261; LCSC Part # (none) -> C190565
Connections:
- net +5V: now also D1.2 (VCC), D2.2 (VCC), D3.2 (VCC), D4.2 (VCC), D5.2 (VCC), D6.2 (VCC), D7.2 (VCC), D8.2 (VCC); no longer D1.1 (VDD), D2.1 (VDD), D3.1 (VDD), D4.1 (VDD), D5.1 (VDD), D6.1 (VDD), D7.1 (VDD), D8.1 (VDD)
- net Dout: now also D8.1 (DOUT); no longer D8.2 (DOUT)
- net at D4.4 (DIN): now also D3.1 (DOUT); no longer D3.2 (DOUT)
- net at D3.4 (DIN): now also D2.1 (DOUT); no longer D2.2 (DOUT)
- net at D5.4 (DIN): now also D4.1 (DOUT); no longer D4.2 (DOUT)
- net at D8.4 (DIN): now also D7.1 (DOUT); no longer D7.2 (DOUT)
- net at D2.4 (DIN): now also D1.1 (DOUT); no longer D1.2 (DOUT)
- net at D6.4 (DIN): now also D5.1 (DOUT); no longer D5.2 (DOUT)
- net at D7.4 (DIN): now also D6.1 (DOUT); no longer D6.2 (DOUT)
